File: E-P-020-R1.0.sch (EAGLE design)
At the start: 25 parts, among them U2 ATMEGA328P_PDIP

Commit message: Added ESC and Encoder
Parts:
- added JP2: ESC_HEADER, SparkFun-Connectors:M03LONGPADS
- added JP3: ENCODER, SparkFun-Connectors:M05PTH
- added R10, R8, R9: 680R, SparkFun-Resistors:0.75OHM-1/4W-1%(0805)
Connections:
- new net ENCODER_A: JP3.5, R10.2, U2.PD2(INT0)
- new net ENCODER_B: JP3.4, R9.2, U2.PD3(INT1)
- new net ENCODER_C: JP3.3, R8.2, U2.PD4(XCK/T0)
- new net ESC_SIG: JP2.3, U2.PD5(T1)
- net +5V: now also JP2.2, JP3.2, R10.1, R8.1, R9.1
- net GND: now also JP2.1, JP3.1
Changed lines of the file:
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@@
 <?xml version="1.0" encoding="utf-8"?>
 <!DOCTYPE eagle SYSTEM "eagle.dtd">
-<eagle version="7.5.0">
+<eagle version="7.3.0">
 <drawing>
 <settings>
@@
 <part name="CAN-BUS" library="adafruit" deviceset="1X4" device="-BIG"/>
 <part name="R7" library="adafruit" deviceset="R-US_" device="M1206"/>
+<part name="JP2" library="SparkFun-Connectors" deviceset="M03" device="LONGPADS" value="ESC_HEADER"/>
+<part name="JP3" library="SparkFun-Connectors" deviceset="M05" device="PTH" value="ENCODER"/>
+<part name="R8" library="SparkFun-Resistors" deviceset="0.75OHM-1/4W-1%(0805)" device="" value="680R"/>
+<part name="R9" library="SparkFun-Resistors" deviceset="0.75OHM-1/4W-1%(0805)" device="" value="680R"/>
+<part name="R10" library="SparkFun-Resistors" deviceset="0.75OHM-1/4W-1%(0805)" device="" value="680R"/>
 </parts>
 <sheets>
@@
 <instance part="CAN-BUS" gate="G$1" x="223.52" y="101.6"/>
 <instance part="R7" gate="G$1" x="198.12" y="101.6" rot="R90"/>
+<instance part="JP2" gate="G$1" x="101.6" y="50.8" rot="R90"/>
+<instance part="JP3" gate="G$1" x="139.7" y="50.8" rot="R90"/>
+<instance part="R8" gate="G$1" x="127" y="86.36"/>
+<instance part="R9" gate="G$1" x="127" y="78.74"/>
+<instance part="R10" gate="G$1" x="127" y="71.12"/>
 </instances>
 <busses>
@@
 <label x="12.7" y="96.52" size="1.778" layer="95"/>
 </segment>
+<segment>
+<pinref part="JP2" gate="G$1" pin="1"/>
+<wire x1="104.14" y1="58.42" x2="104.14" y2="60.96" width="0.1524" layer="91"/>
+<label x="104.14" y="60.96" size="1.778" layer="95" rot="R90"/>
+</segment>
+<segment>
+<pinref part="JP3" gate="G$1" pin="1"/>
+<wire x1="144.78" y1="58.42" x2="144.78" y2="60.96" width="0.1524" layer="91"/>
+<label x="144.78" y="60.96" size="1.778" layer="95" rot="R90"/>
+</segment>
 </net>
 <net name="N$1" class="0">
@@
 <label x="10.16" y="144.78" size="1.778" layer="95"/>
 </segment>
+<segment>
+<pinref part="JP2" gate="G$1" pin="2"/>
+<wire x1="101.6" y1="58.42" x2="101.6" y2="60.96" width="0.1524" layer="91"/>
+<label x="101.6" y="60.96" size="1.778" layer="95" rot="R90"/>
+</segment>
+<segment>
+<pinref part="JP3" gate="G$1" pin="2"/>
+<wire x1="142.24" y1="58.42" x2="142.24" y2="60.96" width="0.1524" layer="91"/>
+<label x="142.24" y="60.96" size="1.778" layer="95" rot="R90"/>
+</segment>
+<segment>
+<pinref part="R8" gate="G$1" pin="1"/>
+<wire x1="121.92" y1="86.36" x2="119.38" y2="86.36" width="0.1524" layer="91"/>
+<wire x1="119.38" y1="86.36" x2="119.38" y2="78.74" width="0.1524" layer="91"/>
+<pinref part="R10" gate="G$1" pin="1"/>
+<wire x1="119.38" y1="78.74" x2="119.38" y2="71.12" width="0.1524" layer="91"/>
+<wire x1="119.38" y1="71.12" x2="121.92" y2="71.12" width="0.1524" layer="91"/>
+<pinref part="R9" gate="G$1" pin="1"/>
+<wire x1="121.92" y1="78.74" x2="119.38" y2="78.74" width="0.1524" layer="91"/>
+<junction x="119.38" y="78.74"/>
+<label x="116.84" y="81.28" size="1.778" layer="95" rot="R270"/>
+</segment>
 </net>
 <net name="OSC1" class="0">
@@
 </segment>
 </net>
+<net name="ESC_SIG" class="0">
+<segment>
+<pinref part="JP2" gate="G$1" pin="3"/>
+<wire x1="99.06" y1="58.42" x2="99.06" y2="60.96" width="0.1524" layer="91"/>
+<label x="99.06" y="60.96" size="1.778" layer="95" rot="R90"/>
+</segment>
+<segment>
+<pinref part="U2" gate="G$1" pin="PD5(T1)"/>
+<wire x1="66.04" y1="114.3" x2="68.58" y2="114.3" width="0.1524" layer="91"/>
+<label x="68.58" y="114.3" size="1.778" layer="95"/>
+</segment>
+</net>
+<net name="ENCODER_A" class="0">
+<segment>
+<pinref part="JP3" gate="G$1" pin="5"/>
+<label x="134.62" y="60.96" size="1.778" layer="95" rot="R90"/>
+<wire x1="134.62" y1="58.42" x2="134.62" y2="71.12" width="0.1524" layer="91"/>
+<pinref part="R10" gate="G$1" pin="2"/>
+<wire x1="134.62" y1="71.12" x2="132.08" y2="71.12" width="0.1524" layer="91"/>
+</segment>
+<segment>
+<pinref part="U2" gate="G$1" pin="PD2(INT0)"/>
+<wire x1="66.04" y1="121.92" x2="68.58" y2="121.92" width="0.1524" layer="91"/>
+<label x="68.58" y="121.92" size="1.778" layer="95"/>
+</segment>
+</net>
+<net name="ENCODER_B" class="0">
+<segment>
+<pinref part="JP3" gate="G$1" pin="4"/>
+<label x="137.16" y="60.96" size="1.778" layer="95" rot="R90"/>
+<pinref part="R9" gate="G$1" pin="2"/>
+<wire x1="132.08" y1="78.74" x2="137.16" y2="78.74" width="0.1524" layer="91"/>
+<wire x1="137.16" y1="78.74" x2="137.16" y2="58.42" width="0.1524" layer="91"/>
+</segment>
+<segment>
+<pinref part="U2" gate="G$1" pin="PD3(INT1)"/>
+<wire x1="66.04" y1="119.38" x2="68.58" y2="119.38" width="0.1524" layer="91"/>
+<label x="68.58" y="119.38" size="1.778" layer="95"/>
+</segment>
+</net>
+<net name="ENCODER_C" class="0">
+<segment>
+<pinref part="JP3" gate="G$1" pin="3"/>
+<label x="139.7" y="60.96" size="1.778" layer="95" rot="R90"/>
+<pinref part="R8" gate="G$1" pin="2"/>
+<wire x1="132.08" y1="86.36" x2="139.7" y2="86.36" width="0.1524" layer="91"/>
+<wire x1="139.7" y1="86.36" x2="139.7" y2="58.42" width="0.1524" layer="91"/>
+</segment>
+<segment>
+<pinref part="U2" gate="G$1" pin="PD4(XCK/T0)"/>
+<wire x1="66.04" y1="116.84" x2="68.58" y2="116.84" width="0.1524" layer="91"/>
+<label x="68.58" y="116.84" size="1.778" layer="95"/>
+</segment>
+</net>
