File: E-P-020-R1.0.sch (EAGLE design)
At the start: 36 parts, among them CN1 1X4-CLEANBIG, J1 1445055-3, U2 ATMEGA328P_PDIP

Commit message: Complete
Parts:
- added LED1, LED2, LED3: (no value), adafruit:LEDSMT1206
- added R11, R12, R13: (no value), E-P-099-R2.2:RESISTOR0805-RES
Connections:
- new net N$10: LED1.C, R11.1
- new net N$11: LED2.C, R12.1
- new net N$12: LED3.C, R13.1
- new net N$6: LED1.A, U2.PC0(ADC0)
- new net N$7: LED2.A, U2.PC1(ADC1)
- new net N$9: LED3.A, U2.PC2(ADC2)
- net GND: now also R11.2, R12.2, R13.2
Changed lines of the file:
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@@
 <part name="C8" library="adafruit" deviceset="C-US" device="C0805"/>
 <part name="C9" library="adafruit" deviceset="C-US" device="C0805"/>
+<part name="LED1" library="adafruit" deviceset="LED" device="SMT1206"/>
+<part name="LED2" library="adafruit" deviceset="LED" device="SMT1206"/>
+<part name="LED3" library="adafruit" deviceset="LED" device="SMT1206"/>
+<part name="R11" library="E-P-099-R2.2" deviceset="RESISTOR" device="0805-RES"/>
+<part name="R12" library="E-P-099-R2.2" deviceset="RESISTOR" device="0805-RES"/>
+<part name="R13" library="E-P-099-R2.2" deviceset="RESISTOR" device="0805-RES"/>
 </parts>
 <sheets>
@@
 <instance part="C8" gate="G$1" x="35.56" y="0" rot="R90"/>
 <instance part="C9" gate="G$1" x="35.56" y="-7.62" rot="R90"/>
+<instance part="LED1" gate="G$1" x="71.12" y="149.86" rot="R90"/>
+<instance part="LED2" gate="G$1" x="71.12" y="147.32" rot="R90"/>
+<instance part="LED3" gate="G$1" x="71.12" y="144.78" rot="R90"/>
+<instance part="R11" gate="G$1" x="81.28" y="149.86"/>
+<instance part="R12" gate="G$1" x="81.28" y="147.32"/>
+<instance part="R13" gate="G$1" x="81.28" y="144.78"/>
 </instances>
 <busses>
@@
 <junction x="33.02" y="0"/>
 <pinref part="C9" gate="G$1" pin="1"/>
+</segment>
+<segment>
+<pinref part="R11" gate="G$1" pin="2"/>
+<pinref part="R12" gate="G$1" pin="2"/>
+<wire x1="86.36" y1="149.86" x2="86.36" y2="147.32" width="0.1524" layer="91"/>
+<pinref part="R13" gate="G$1" pin="2"/>
+<wire x1="86.36" y1="147.32" x2="86.36" y2="144.78" width="0.1524" layer="91"/>
+<junction x="86.36" y="147.32"/>
+<label x="86.36" y="147.32" size="1.778" layer="95"/>
 </segment>
 </net>
@@
 </segment>
 </net>
+<net name="N$6" class="0">
+<segment>
+<pinref part="U2" gate="G$1" pin="PC0(ADC0)"/>
+<pinref part="LED1" gate="G$1" pin="A"/>
+<wire x1="66.04" y1="149.86" x2="68.58" y2="149.86" width="0.1524" layer="91"/>
+</segment>
+</net>
+<net name="N$7" class="0">
+<segment>
+<pinref part="U2" gate="G$1" pin="PC1(ADC1)"/>
+<pinref part="LED2" gate="G$1" pin="A"/>
+<wire x1="66.04" y1="147.32" x2="68.58" y2="147.32" width="0.1524" layer="91"/>
+</segment>
+</net>
+<net name="N$9" class="0">
+<segment>
+<pinref part="U2" gate="G$1" pin="PC2(ADC2)"/>
+<pinref part="LED3" gate="G$1" pin="A"/>
+<wire x1="66.04" y1="144.78" x2="68.58" y2="144.78" width="0.1524" layer="91"/>
+</segment>
+</net>
+<net name="N$10" class="0">
+<segment>
+<pinref part="LED1" gate="G$1" pin="C"/>
+<pinref part="R11" gate="G$1" pin="1"/>
+</segment>
+</net>
+<net name="N$11" class="0">
+<segment>
+<pinref part="LED2" gate="G$1" pin="C"/>
+<pinref part="R12" gate="G$1" pin="1"/>
+</segment>
+</net>
+<net name="N$12" class="0">
+<segment>
+<pinref part="LED3" gate="G$1" pin="C"/>
+<pinref part="R13" gate="G$1" pin="1"/>
+</segment>
+</net>

Commit message: Update
Connections:
- removed net CEN2: U2.PB0(ICP)
Changed lines of the file:
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@@
 <pinref part="U2" gate="G$1" pin="GND@1"/>
 <wire x1="17.78" y1="96.52" x2="15.24" y2="96.52" width="0.1524" layer="91"/>
+<label x="12.7" y="96.52" size="1.778" layer="95"/>
 <pinref part="U2" gate="G$1" pin="GND@2"/>
+<wire x1="15.24" y1="96.52" x2="12.7" y2="96.52" width="0.1524" layer="91"/>
 <wire x1="17.78" y1="93.98" x2="15.24" y2="93.98" width="0.1524" layer="91"/>
 <wire x1="15.24" y1="93.98" x2="15.24" y2="96.52" width="0.1524" layer="91"/>
-<wire x1="15.24" y1="96.52" x2="12.7" y2="96.52" width="0.1524" layer="91"/>
-<label x="12.7" y="96.52" size="1.778" layer="95"/>
+<junction x="15.24" y="96.52"/>
 </segment>
 <segment>
@@
 <pinref part="U2" gate="G$1" pin="AVCC"/>
 <wire x1="17.78" y1="144.78" x2="15.24" y2="144.78" width="0.1524" layer="91"/>
+<label x="10.16" y="144.78" size="1.778" layer="95"/>
 <pinref part="U2" gate="G$1" pin="VCC"/>
+<wire x1="15.24" y1="144.78" x2="12.7" y2="144.78" width="0.1524" layer="91"/>
 <wire x1="17.78" y1="142.24" x2="15.24" y2="142.24" width="0.1524" layer="91"/>
 <wire x1="15.24" y1="142.24" x2="15.24" y2="144.78" width="0.1524" layer="91"/>
-<wire x1="15.24" y1="144.78" x2="12.7" y2="144.78" width="0.1524" layer="91"/>
-<label x="10.16" y="144.78" size="1.778" layer="95"/>
+<junction x="15.24" y="144.78"/>
 </segment>
 <segment>
@@
 </segment>
 </net>
-<net name="CEN2" class="0">
-<segment>
-<pinref part="U2" gate="G$1" pin="PB0(ICP)"/>
-<wire x1="66.04" y1="104.14" x2="68.58" y2="104.14" width="0.1524" layer="91"/>
-</segment>
-</net>
