File: E-P-020-R1.0.brd (EAGLE design)
At the start: 50 x 50 mm, 36 parts, among them CN1 1X4-CLEANBIG, J1 1445055-3, U2 ATMEGA328P_PDIP

Commit message: Complete
Parts:
- added LED1, LED2, LED3: (no value), adafruit:1206
- added R11, R12, R13: (no value), E-P-099-R2.2:0805
- moved R2 0.50 mm to (20.3, 35.9)
Connections:
- new net N$10: LED1.C, R11.1
- new net N$11: LED2.C, R12.1
- new net N$12: LED3.C, R13.1
- new net N$6: LED1.A, U2.23
- new net N$7: LED2.A, U2.24
- new net N$9: LED3.A, U2.25
- net GND: now also R11.2, R12.2, R13.2
Routing:
- net N$7: track 0.00 -> 3.49 mm
- net N$9: track 0.00 -> 3.31 mm
- net N$6: track 0.00 -> 3.21 mm
- net N$12: track 0.00 -> 2.99 mm
- net N$11: track 0.00 -> 2.95 mm
- net N$10: track 0.00 -> 2.45 mm
- net N$8: track 0.53 -> 2.41 mm
- net +5V: track 153.4 -> 154.4 mm
- net N$2: track 3.00 -> 2.50 mm
Changed lines of the file:
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@@
 <attribute name="NAME" x="22.9555" y="11.812" size="1" layer="25" rot="R270"/>
 </element>
-<element name="R2" library="SparkFun-Passives" package="0805" value="" x="20.34" y="35.44" smashed="yes" rot="R180">
-<attribute name="NAME" x="21.102" y="34.6145" size="1" layer="25" rot="R180"/>
-<attribute name="VALUE" x="21.356" y="36.837" size="0.4064" layer="27" rot="R180"/>
+<element name="R2" library="SparkFun-Passives" package="0805" value="" x="20.34" y="35.94" smashed="yes" rot="R180">
+<attribute name="NAME" x="23.602" y="36.5145" size="1" layer="25" rot="R180"/>
+<attribute name="VALUE" x="21.356" y="37.337" size="0.4064" layer="27" rot="R180"/>
 </element>
 <element name="R3" library="SparkFun-Passives" package="0805" value="" x="13.35" y="17.14" smashed="yes" rot="R180">
@@
 </element>
 <element name="R4" library="SparkFun-Passives" package="0805" value="" x="12.54" y="37.06" smashed="yes">
-<attribute name="NAME" x="14.778" y="36.4855" size="1" layer="25"/>
+<attribute name="NAME" x="9.378" y="36.7855" size="1" layer="25"/>
 <attribute name="VALUE" x="11.524" y="35.663" size="0.4064" layer="27"/>
 </element>
@@
 <attribute name="NAME" x="1.684" y="16.211" size="1" layer="25" rot="R90"/>
 <attribute name="VALUE" x="3.786" y="19.011" size="1.27" layer="27" rot="R90"/>
+</element>
+<element name="LED1" library="adafruit" package="1206" value="" x="21.1" y="32.5" smashed="yes" rot="R90">
+<attribute name="NAME" x="20.33" y="28.43" size="1" layer="25" rot="R90"/>
+<attribute name="VALUE" x="23.64" y="31.23" size="1.27" layer="27" rot="R90"/>
+</element>
+<element name="LED2" library="adafruit" package="1206" value="" x="18.5" y="32.8" smashed="yes" rot="R90">
+<attribute name="NAME" x="17.73" y="28.23" size="1" layer="25" rot="R90"/>
+<attribute name="VALUE" x="21.04" y="31.53" size="1.27" layer="27" rot="R90"/>
+</element>
+<element name="LED3" library="adafruit" package="1206" value="" x="15.9" y="32.6" smashed="yes" rot="R90">
+<attribute name="NAME" x="15.03" y="28.23" size="1" layer="25" rot="R90"/>
+<attribute name="VALUE" x="18.44" y="31.33" size="1.27" layer="27" rot="R90"/>
+</element>
+<element name="R11" library="E-P-099-R2.2" package="0805" value="" x="23.5" y="32.9" smashed="yes" rot="R270">
+<attribute name="NAME" x="24.3255" y="33.662" size="1" layer="25" rot="R270"/>
+<attribute name="VALUE" x="20.833" y="33.916" size="1.27" layer="27" rot="R270"/>
+</element>
+<element name="R12" library="E-P-099-R2.2" package="0805" value="" x="16.7" y="36.8" smashed="yes" rot="R180">
+<attribute name="NAME" x="17.562" y="38.6745" size="1" layer="25" rot="R180"/>
+<attribute name="VALUE" x="17.716" y="39.467" size="1.27" layer="27" rot="R180"/>
+</element>
+<element name="R13" library="E-P-099-R2.2" package="0805" value="" x="12.6" y="32.6" smashed="yes" rot="R180">
+<attribute name="NAME" x="13.662" y="31.6745" size="1" layer="25" rot="R180"/>
+<attribute name="VALUE" x="13.616" y="35.267" size="1.27" layer="27" rot="R180"/>
 </element>
 </elements>
@@
 <via x="29.8" y="24" extent="1-16" drill="0.4"/>
 <via x="23.3" y="25.3" extent="1-16" drill="0.4"/>
-<via x="15.9" y="25.2" extent="1-16" drill="0.4"/>
+<via x="16.1" y="25.5" extent="1-16" drill="0.4"/>
 <via x="11" y="25.1" extent="1-16" drill="0.4"/>
-<via x="11.9" y="32.8" extent="1-16" drill="0.4"/>
-<via x="20.4" y="31.8" extent="1-16" drill="0.4"/>
+<via x="10.3" y="32.6" extent="1-16" drill="0.4"/>
+<via x="22.7" y="30.5" extent="1-16" drill="0.4"/>
 <via x="27.7" y="35.2" extent="1-16" drill="0.4"/>
 <via x="30" y="31.5" extent="1-16" drill="0.4"/>
@@
 <via x="9.1" y="44.3" extent="1-16" drill="0.4"/>
 <via x="9.6" y="38.4" extent="1-16" drill="0.4"/>
+<contactref element="R11" pad="2"/>
+<contactref element="R12" pad="2"/>
+<contactref element="R13" pad="2"/>
 </signal>
 <signal name="N$1">
@@
 <wire x1="4.6" y1="22.5" x2="4" y2="22.5" width="0.4064" layer="1"/>
 <wire x1="4" y1="22.5" x2="2.455" y2="24.045" width="0.4064" layer="1"/>
-<wire x1="19.25" y1="24.6" x2="19.25" y2="24.65" width="0.4064" layer="1"/>
-<wire x1="19.25" y1="24.65" x2="17.4" y2="26.5" width="0.4064" layer="1"/>
-<wire x1="17.4" y1="26.5" x2="17.4" y2="28.8" width="0.4064" layer="1"/>
-<wire x1="17.4" y1="28.8" x2="15.1" y2="31.1" width="0.4064" layer="1"/>
-<wire x1="15.1" y1="31.1" x2="5.22" y2="31.1" width="0.4064" layer="1"/>
+<wire x1="5.22" y1="31.1" x2="12.9" y2="31.1" width="0.4064" layer="1"/>
+<wire x1="12.9" y1="31.1" x2="14.7" y2="29.3" width="0.4064" layer="1"/>
+<wire x1="14.7" y1="29.3" x2="14.7" y2="25.2" width="0.4064" layer="1"/>
+<wire x1="14.7" y1="25.2" x2="15.3" y2="24.6" width="0.4064" layer="1"/>
+<wire x1="15.3" y1="24.6" x2="19.25" y2="24.6" width="0.4064" layer="1"/>
 </signal>
 <signal name="OSC1">
@@
 <contactref element="U$2" pad="8"/>
 <contactref element="R2" pad="2"/>
-<wire x1="18.85" y1="38.2" x2="18.85" y2="36.03" width="0.4064" layer="1"/>
-<wire x1="18.85" y1="36.03" x2="19.44" y2="35.44" width="0.4064" layer="1"/>
+<wire x1="19.44" y1="35.94" x2="19.44" y2="37.61" width="0.4064" layer="1"/>
+<wire x1="19.44" y1="37.61" x2="18.85" y2="38.2" width="0.4064" layer="1"/>
 </signal>
 <signal name="TX">
@@
 <contactref element="PWR" pad="C"/>
 <wire x1="5.1" y1="25.32" x2="5.13" y2="25.85" width="0.4064" layer="1"/>
-<wire x1="5.13" y1="25.85" x2="5.1" y2="27.72" width="0" layer="19" extent="1-1"/>
+<wire x1="5.13" y1="25.85" x2="5.13" y2="27.69" width="0.4064" layer="1"/>
+<wire x1="5.13" y1="27.69" x2="5.1" y2="27.72" width="0.4064" layer="1"/>
 </signal>
 <signal name="CEN2">
@@
 <wire x1="12.1" y1="5.92" x2="12.1" y2="21.4" width="0.254" layer="16"/>
 </signal>
+<signal name="N$6">
+<contactref element="U2" pad="23"/>
+<contactref element="LED1" pad="A"/>
+<wire x1="21.04" y1="27.89" x2="21.04" y2="31.018" width="0.4064" layer="1"/>
+<wire x1="21.04" y1="31.018" x2="21.1" y2="31.078" width="0.4064" layer="1"/>
+</signal>
+<signal name="N$7">
+<contactref element="U2" pad="24"/>
+<contactref element="LED2" pad="A"/>
+<wire x1="18.5" y1="27.89" x2="18.5" y2="31.378" width="0.4064" layer="1"/>
+</signal>
+<signal name="N$9">
+<contactref element="U2" pad="25"/>
+<contactref element="LED3" pad="A"/>
+<wire x1="15.96" y1="27.89" x2="15.96" y2="31.118" width="0.4064" layer="1"/>
+<wire x1="15.96" y1="31.118" x2="15.9" y2="31.178" width="0.4064" layer="1"/>
+</signal>
+<signal name="N$10">
+<contactref element="LED1" pad="C"/>
+<contactref element="R11" pad="1"/>
+<wire x1="21.1" y1="33.922" x2="23.378" y2="33.922" width="0.4064" layer="1"/>
+<wire x1="23.378" y1="33.922" x2="23.5" y2="33.8" width="0.4064" layer="1"/>
+</signal>
+<signal name="N$11">
+<contactref element="LED2" pad="C"/>
+<contactref element="R12" pad="1"/>
+<wire x1="18.5" y1="34.222" x2="18.5" y2="35.9" width="0.4064" layer="1"/>
+<wire x1="18.5" y1="35.9" x2="17.6" y2="36.8" width="0.4064" layer="1"/>
+</signal>
+<signal name="N$12">
+<contactref element="LED3" pad="C"/>
+<contactref element="R13" pad="1"/>
+<wire x1="15.9" y1="34.022" x2="14.922" y2="34.022" width="0.4064" layer="1"/>
+<wire x1="14.922" y1="34.022" x2="13.5" y2="32.6" width="0.4064" layer="1"/>
+</signal>
 </signals>

Commit message: Update
Connections:
- removed net CEN2: U2.14
Changed lines of the file:
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@@
 <contactref element="C7" pad="2"/>
 <contactref element="U2" pad="8"/>
-<contactref element="U2" pad="22"/>
 <polygon width="0.4064" layer="16">
 <vertex x="59" y="56.5"/>
@@
 <contactref element="R12" pad="2"/>
 <contactref element="R13" pad="2"/>
+<contactref element="U2" pad="22"/>
 </signal>
 <signal name="N$1">
@@
 <contactref element="PWR" pad="A"/>
 <contactref element="U2" pad="20"/>
-<contactref element="U2" pad="7"/>
 <contactref element="R8" pad="1"/>
 <contactref element="R10" pad="1"/>
 <contactref element="R9" pad="1"/>
-<wire x1="23.58" y1="20.27" x2="23.58" y2="18.58" width="0.4064" layer="1"/>
 <wire x1="23.58" y1="18.58" x2="22.1" y2="17.1" width="0.4064" layer="1"/>
 <wire x1="22.1" y1="17.1" x2="21.4" y2="17.1" width="0.4064" layer="1"/>
 <wire x1="21.4" y1="17.1" x2="14.29" y2="17.1" width="0.4064" layer="1"/>
 <wire x1="14.29" y1="17.1" x2="14.25" y2="17.14" width="0.4064" layer="1"/>
-<wire x1="23.58" y1="20.27" x2="23.58" y2="20.38" width="0.4064" layer="1"/>
 <wire x1="23.58" y1="20.38" x2="28.7" y2="25.5" width="0.4064" layer="1"/>
 <wire x1="28.7" y1="25.5" x2="28.7" y2="27.85" width="0.4064" layer="1"/>
@@
 <contactref element="U2" pad="21"/>
 <wire x1="5.01" y1="39.13" x2="5.01" y2="31.31" width="0.4064" layer="1"/>
-<wire x1="19.25" y1="24.6" x2="23.58" y2="20.27" width="0.4064" layer="1"/>
 <wire x1="28.66" y1="27.89" x2="26.12" y2="27.89" width="0.4064" layer="1"/>
 <wire x1="26.12" y1="27.89" x2="26.12" y2="32.58" width="0.4064" layer="1"/>
@@
 <wire x1="14.7" y1="25.2" x2="15.3" y2="24.6" width="0.4064" layer="1"/>
 <wire x1="15.3" y1="24.6" x2="19.25" y2="24.6" width="0.4064" layer="1"/>
+<contactref element="U2" pad="7"/>
+<wire x1="19.25" y1="24.6" x2="23.58" y2="20.27" width="0.4064" layer="1"/>
+<wire x1="23.58" y1="20.27" x2="23.58" y2="18.58" width="0.4064" layer="1"/>
+<wire x1="23.58" y1="20.38" x2="23.58" y2="20.27" width="0.4064" layer="1"/>
 </signal>
 <signal name="OSC1">
@@
 <wire x1="5.13" y1="27.69" x2="5.1" y2="27.72" width="0.4064" layer="1"/>
 </signal>
-<signal name="CEN2">
-<contactref element="U2" pad="14"/>
-</signal>
 <signal name="ESC_SIG">
