File: R2.0/E-P-020-R2.0.brd (EAGLE design)
At the start: 48.6 x 47.6 mm, 21 parts, among them J1 1445055-3

Commit message: Added version number to board
Parts:
- moved U$4 4.49 mm to (15.2, 38.1)
Other:
- board text added: "E-P-020-R2.0"
Changed lines of the file:
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@@
 <?xml version="1.0" encoding="utf-8"?>
 <!DOCTYPE eagle SYSTEM "eagle.dtd">
-<eagle version="7.3.0">
+<eagle version="7.5.0">
 <drawing>
 <settings>
@@
 <wire x1="48.565" y1="51.425" x2="0" y2="51.425" width="0" layer="20"/>
 <wire x1="0" y1="51.425" x2="0" y2="3.81" width="0" layer="20"/>
+<text x="8.255" y="33.02" size="1.778" layer="21">E-P-020-R2.0</text>
 </plain>
 <attributes>
@@
 </element>
 <element name="U$3" library="Shell2015" package="CAN_6P6C" value="CAN_6P6C" x="6.35" y="11.43"/>
-<element name="U$4" library="Shell2015" package="LOGO" value="LOGO" x="10.795" y="37.465"/>
+<element name="U$4" library="Shell2015" package="LOGO" value="LOGO" x="15.24" y="38.1"/>
 <element name="U$5" library="Shell2015" package="CAN_6P6C" value="CAN_6P6C" x="21.59" y="11.43"/>
 </elements>
