File: R1.0/E-P-020-R1.0.brd (EAGLE design)
At the start: 50 x 50 mm, 42 parts, among them CN1 1X4-CLEANBIG, J1 1445055-3, U2 ATMEGA328P_PDIP

Commit message: Added resistor/capacitor values
Parts:
- C1, C2, C3, C4: value (none) -> 18pf
- C5, C9: value (none) -> 0.1uf
- C8: value (none) -> 10uf
- R1, R11, R12, R13, R2, R3, R6: value (none) -> 1k
- R7: value (none) -> 120
Changed lines of the file:
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@@
 </autorouter>
 <elements>
-<element name="C1" library="SparkFun-Capacitors" package="0805" value="" x="29.66" y="45.34" smashed="yes" rot="R180">
+<element name="C1" library="SparkFun-Capacitors" package="0805" value="18pf" x="29.66" y="45.34" smashed="yes" rot="R180">
 <attribute name="NAME" x="30.422" y="44.5145" size="1" layer="25" rot="R180"/>
 <attribute name="VALUE" x="30.676" y="46.737" size="0.4064" layer="27" rot="R180"/>
 </element>
-<element name="C2" library="SparkFun-Capacitors" package="0805" value="" x="38.23" y="45.06" smashed="yes">
+<element name="C2" library="SparkFun-Capacitors" package="0805" value="18pf" x="38.23" y="45.06" smashed="yes">
 <attribute name="NAME" x="37.468" y="45.8855" size="1" layer="25"/>
 <attribute name="VALUE" x="37.214" y="43.663" size="0.4064" layer="27"/>
 </element>
-<element name="C3" library="SparkFun-Capacitors" package="0805" value="" x="25.18" y="15.74" smashed="yes" rot="R180">
+<element name="C3" library="SparkFun-Capacitors" package="0805" value="18pf" x="25.18" y="15.74" smashed="yes" rot="R180">
 <attribute name="NAME" x="25.942" y="14.9145" size="1" layer="25" rot="R180"/>
 <attribute name="VALUE" x="26.196" y="17.137" size="0.4064" layer="27" rot="R180"/>
 </element>
-<element name="C4" library="SparkFun-Capacitors" package="0805" value="" x="34.71" y="15.86" smashed="yes">
+<element name="C4" library="SparkFun-Capacitors" package="0805" value="18pf" x="34.71" y="15.86" smashed="yes">
 <attribute name="NAME" x="33.948" y="16.6855" size="1" layer="25"/>
 <attribute name="VALUE" x="33.694" y="14.463" size="0.4064" layer="27"/>
 </element>
-<element name="C5" library="SparkFun-Capacitors" package="0805" value="" x="13.3" y="14.54" smashed="yes" rot="R180">
+<element name="C5" library="SparkFun-Capacitors" package="0805" value="0.1uf" x="13.3" y="14.54" smashed="yes" rot="R180">
 <attribute name="NAME" x="14.062" y="13.7145" size="1" layer="25" rot="R180"/>
 <attribute name="VALUE" x="14.316" y="15.937" size="0.4064" layer="27" rot="R180"/>
@@
 <attribute name="VALUE" x="2.56" y="30.74" size="1.27" layer="27" rot="R270"/>
 </element>
-<element name="R1" library="SparkFun-Passives" package="0805" value="" x="44.96" y="31.03" smashed="yes" rot="R270">
+<element name="R1" library="SparkFun-Passives" package="0805" value="1k" x="44.96" y="31.03" smashed="yes" rot="R270">
 <attribute name="NAME" x="45.7855" y="31.792" size="1" layer="25" rot="R270"/>
 <attribute name="VALUE" x="43.563" y="32.046" size="0.4064" layer="27" rot="R270"/>
@@
 <attribute name="NAME" x="22.9555" y="11.812" size="1" layer="25" rot="R270"/>
 </element>
-<element name="R2" library="SparkFun-Passives" package="0805" value="" x="20.34" y="35.94" smashed="yes" rot="R180">
+<element name="R2" library="SparkFun-Passives" package="0805" value="1k" x="20.34" y="35.94" smashed="yes" rot="R180">
 <attribute name="NAME" x="23.602" y="36.5145" size="1" layer="25" rot="R180"/>
 <attribute name="VALUE" x="21.356" y="37.337" size="0.4064" layer="27" rot="R180"/>
 </element>
-<element name="R3" library="SparkFun-Passives" package="0805" value="" x="13.35" y="17.14" smashed="yes" rot="R180">
+<element name="R3" library="SparkFun-Passives" package="0805" value="1k" x="13.35" y="17.14" smashed="yes" rot="R180">
 <attribute name="NAME" x="14.112" y="16.3145" size="1" layer="25" rot="R180"/>
 <attribute name="VALUE" x="14.366" y="18.537" size="0.4064" layer="27" rot="R180"/>
@@
 <attribute name="VALUE" x="11.773" y="45.956" size="0.4064" layer="27" rot="R270"/>
 </element>
-<element name="R6" library="SparkFun-Passives" package="0805" value="" x="5.13" y="24.95" smashed="yes" rot="R90">
+<element name="R6" library="SparkFun-Passives" package="0805" value="1k" x="5.13" y="24.95" smashed="yes" rot="R90">
 <attribute name="NAME" x="7.4045" y="23.988" size="1" layer="25" rot="R90"/>
 <attribute name="VALUE" x="6.527" y="23.934" size="0.4064" layer="27" rot="R90"/>
 </element>
-<element name="R7" library="adafruit" package="M1206" value="" x="13.27" y="40.85" smashed="yes" rot="R90">
+<element name="R7" library="adafruit" package="M1206" value="120" x="13.27" y="40.85" smashed="yes" rot="R90">
 <attribute name="NAME" x="16.1" y="40.18" size="1" layer="25" rot="R90"/>
 <attribute name="VALUE" x="15.81" y="39.58" size="1.27" layer="27" rot="R90"/>
@@
 </element>
 <element name="3.3V_REG" library="mylibrary" package="SOT-23A" value="MCP1702" x="4.6" y="22.5" smashed="yes"/>
-<element name="C8" library="adafruit" package="C0805" value="" x="2" y="5.1" smashed="yes" rot="R90">
+<element name="C8" library="adafruit" package="C0805" value="10uf" x="2" y="5.1" smashed="yes" rot="R90">
 <attribute name="NAME" x="0.984" y="4.211" size="1" layer="25" rot="R90"/>
 <attribute name="VALUE" x="4.286" y="4.211" size="1.27" layer="27" rot="R90"/>
 </element>
-<element name="C9" library="adafruit" package="C0805" value="" x="1.5" y="19.9" smashed="yes" rot="R90">
+<element name="C9" library="adafruit" package="C0805" value="0.1uf" x="1.5" y="19.9" smashed="yes" rot="R90">
 <attribute name="NAME" x="1.684" y="16.211" size="1" layer="25" rot="R90"/>
 <attribute name="VALUE" x="3.786" y="19.011" size="1.27" layer="27" rot="R90"/>
@@
 <attribute name="VALUE" x="18.44" y="31.33" size="1.27" layer="27" rot="R90"/>
 </element>
-<element name="R11" library="E-P-099-R2.2" package="0805" value="" x="23.5" y="32.9" smashed="yes" rot="R270">
+<element name="R11" library="E-P-099-R2.2" package="0805" value="1k" x="23.5" y="32.9" smashed="yes" rot="R270">
 <attribute name="NAME" x="24.3255" y="33.662" size="1" layer="25" rot="R270"/>
 <attribute name="VALUE" x="20.833" y="33.916" size="1.27" layer="27" rot="R270"/>
 </element>
-<element name="R12" library="E-P-099-R2.2" package="0805" value="" x="16.7" y="36.8" smashed="yes" rot="R180">
+<element name="R12" library="E-P-099-R2.2" package="0805" value="1k" x="16.7" y="36.8" smashed="yes" rot="R180">
 <attribute name="NAME" x="17.562" y="38.6745" size="1" layer="25" rot="R180"/>
 <attribute name="VALUE" x="17.716" y="39.467" size="1.27" layer="27" rot="R180"/>
 </element>
-<element name="R13" library="E-P-099-R2.2" package="0805" value="" x="12.6" y="32.6" smashed="yes" rot="R180">
+<element name="R13" library="E-P-099-R2.2" package="0805" value="1k" x="12.6" y="32.6" smashed="yes" rot="R180">
 <attribute name="NAME" x="13.662" y="31.6745" size="1" layer="25" rot="R180"/>
 <attribute name="VALUE" x="13.616" y="35.267" size="1.27" layer="27" rot="R180"/>
