File: R1.0/E-P-020-R1.0.brd (EAGLE design)
At the start: 50 x 50 mm, 42 parts, among them CN1 1X4-CLEANBIG, J1 1445055-3, U2 ATMEGA328P_PDIP

Commit message: Integrated pedal, started working on the current sensor
Parts:
- R3: value 1k -> 10k
Changed lines of the file:
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@@
 <attribute name="VALUE" x="21.356" y="37.337" size="0.4064" layer="27" rot="R180"/>
 </element>
-<element name="R3" library="SparkFun-Passives" package="0805" value="1k" x="13.35" y="17.14" smashed="yes" rot="R180">
+<element name="R3" library="SparkFun-Passives" package="0805" value="10k" x="13.35" y="17.14" smashed="yes" rot="R180">
 <attribute name="NAME" x="14.112" y="16.3145" size="1" layer="25" rot="R180"/>
 <attribute name="VALUE" x="14.366" y="18.537" size="0.4064" layer="27" rot="R180"/>
